File: hardware/4in1.kicad_sch (KiCad schematic)
At the start: 29 parts, among them J1 SM08B-SRSS-TB, U12 INA186A3IDCKR, U13 LMR54406DBVR, U14 FTC160808S4R7MBCA, U15 TLV76733DRVR

Commit message: Fix JLCPCB placement offsets in the toolkit config (#43)
Mirror of OpenESC-20x20 #45. AUTO TRANSLATE applied the toolkit's
generic QFN (+90) and SOT-23/SOT-363 (+180) rules to EasyEDA-derived
footprints that already match the JLCPCB library. Disable it and set
explicit offsets measured against the EasyEDA footprints:

- U12 (C2058245): FT Rotation Offset 270
- Q1-Q24 (C22385416): FT Position Offset 0,-1.06
- J1 (C160407): FT Position Offset 0,2.835

Metadata only: netlist differs by the new fields, ERC/DRC unchanged.

Co-authored-by: Claude Opus 5.5 <noreply@anthropic.com>
Parts:
- J1: FT Position Offset (none) -> 0,2.835
- U12: FT Rotation Offset (none) -> 270
