File: hardware/ESC.kicad_sch (KiCad schematic)
At the start: 36 parts, among them Q1 SP40N01GHNK, Q11 SP40N01GHNK, Q16 SP40N01GHNK, Q2 SP40N01GHNK, Q21 SP40N01GHNK, Q6 SP40N01GHNK, U2 AT32F421G8U7, U4 NSG2065Q

Commit message: Fix JLCPCB placement offsets in the toolkit config (#43)
Mirror of OpenESC-20x20 #45. AUTO TRANSLATE applied the toolkit's
generic QFN (+90) and SOT-23/SOT-363 (+180) rules to EasyEDA-derived
footprints that already match the JLCPCB library. Disable it and set
explicit offsets measured against the EasyEDA footprints:

- U12 (C2058245): FT Rotation Offset 270
- Q1-Q24 (C22385416): FT Position Offset 0,-1.06
- J1 (C160407): FT Position Offset 0,2.835

Metadata only: netlist differs by the new fields, ERC/DRC unchanged.

Co-authored-by: Claude Opus 5.5 <noreply@anthropic.com>
Parts:
- Q1, Q11, Q16, Q2, Q21, Q6: FT Position Offset (none) -> 0,-1.06
